Commit message: UPDATE map and robot urdf empty track map added and robot gazebo and urdf file updated

File: vehicle_sim/urdf/ackermann.gazebo.xacro (robot description, xacro)
@@ -61,12 +61,12 @@
     <gazebo reference="camera_link">
         <sensor name="depth_camera" type="rgbd_camera">
-            <topic>depth_camera</topic>
+            <topic>camera</topic>
             <ignition_frame_id>camera_link</ignition_frame_id>
             <always_on>true</always_on>
-            <visualize>false</visualize>
+            <visualize>true</visualize>
             <update_rate>5.0</update_rate>
             <frame_id>camera_link</frame_id>
             <camera>
-            <horizontal_fov>1.047198</horizontal_fov>
+            <horizontal_fov>1.085595</horizontal_fov>
             <image>
                 <width>640</width>
@@ -75,5 +75,5 @@
             <clip>
                 <near>0.05</near>
-                <far>3</far>
+                <far>8</far>
             </clip>
             </camera>

File: vehicle_sim/urdf/ackermann.urdf.xacro (robot description, xacro)
@@ -202,5 +202,5 @@
     </link>
     <joint name="lidar_link_joint" type="fixed">
-        <origin xyz="0.0 0.0 0.175" rpy="0.0 -0.0 0.0" />
+        <origin xyz="0.4 0.0 0.175" rpy="0.0 -0.0 0.0" />
         <parent link="base_link" />
         <child link="lidar_link" />
@@ -215,5 +215,5 @@
             <origin xyz="0.0 0.0 0.0" rpy="0.0 0.0 0.0"/>
             <geometry>
-                <cylinder radius="0.05" length="0.1"/>
+                <cylinder radius="0.05" length="0.3"/>
             </geometry>
             <material name="camera">
@@ -229,5 +229,5 @@
     </link>
     <joint name="camera_link_joint" type="fixed">
-        <origin xyz="0.0 0.0 0.24" rpy="0.0 0.0 0.0" />
+        <origin xyz="0.4 0.0 0.24" rpy="0.0 0.0 0.0" />
         <parent link="base_link" />
         <child link="camera_link" />

Commit message: UPDATE robot lidar robot lidar position changed and scan angle seted for wheel and front distance

File: vehicle_sim/urdf/ackermann.gazebo.xacro (robot description, xacro)
@@ -19,6 +19,6 @@
                         <samples>270</samples>
                         <resolution>1.0</resolution>
-                        <min_angle>-2.35619</min_angle>
-                        <max_angle>2.35619</max_angle>
+                        <min_angle>-1.435096</min_angle>
+                        <max_angle>1.435096</max_angle>
                     </horizontal>
                 </scan>

File: vehicle_sim/urdf/ackermann.urdf.xacro (robot description, xacro)
@@ -202,5 +202,5 @@
     </link>
     <joint name="lidar_link_joint" type="fixed">
-        <origin xyz="0.4 0.0 0.175" rpy="0.0 -0.0 0.0" />
+        <origin xyz="0.5 0.0 -0.160" rpy="0.0 -0.0 0.0" />
         <parent link="base_link" />
         <child link="lidar_link" />
