Commit message: UPDATE vehicle simulation launch file vehicle simulation launch file connected other launch file and lidar position changed

File: vehicle_sim/urdf/ackermann.urdf.xacro (robot description, xacro)
@@ -188,5 +188,5 @@
             <origin xyz="0.0 0.0 0.0" rpy="0.0 0.0 0.0"/>
             <geometry>
-                 <cylinder radius="0.075" length="0.05"/>
+                 <cylinder radius="0.075" length="0.03"/>
             </geometry>
             <material name="lidar_blue">
@@ -197,10 +197,10 @@
             <origin xyz="0.0 0.0 0.0" rpy="0.0 0.0 0.0"/>
             <geometry>
-                <cylinder radius="0.075" length="0.05"/>
+                <cylinder radius="0.075" length="0.03"/>
             </geometry>
         </collision>
     </link>
     <joint name="lidar_link_joint" type="fixed">
-        <origin xyz="0.5 0.0 -0.160" rpy="0.0 -0.0 0.0" />
+        <origin xyz="0.5 0.0 -0.150" rpy="0.0 -0.0 0.0" />
         <parent link="base_link" />
         <child link="lidar_link" />

Commit message: ADD racing lap mode amcl and nav2 inculed racing mode is working

File: vehicle_sim/urdf/ackermann.urdf.xacro (robot description, xacro)
@@ -201,7 +201,38 @@
         </collision>
     </link>
+    <!-- Lidar Mounting Bracket (Aracın önüne uzanan kol) -->
+    <link name="lidar_mount_link">
+        <inertial>
+            <origin xyz="0.0 0.0 0.0" rpy="0.0 0.0 0.0"/>
+            <mass value="0.1"/>
+            <inertia ixx="0.001" ixy="0.0" ixz="0.0" iyy="0.001" iyz="0.0" izz="0.001"/>
+        </inertial>
+        <visual>
+            <origin xyz="0.125 0.0 0.0" rpy="0.0 0.0 0.0"/>
+            <geometry>
+                <!-- 25cm uzunluğunda, 3cm kalınlığında kol -->
+                <box size="0.25 0.03 0.03"/>
+            </geometry>
+            <material name="mount_gray">
+                <color rgba="0.4 0.4 0.4 1"/>
+            </material>
+        </visual>
+        <collision>
+            <origin xyz="0.125 0.0 0.0" rpy="0.0 0.0 0.0"/>
+            <geometry>
+                <box size="0.25 0.03 0.03"/>
+            </geometry>
+        </collision>
+    </link>
+    <joint name="lidar_mount_joint" type="fixed">
+        <!-- Bracket base_link'in önünden başlıyor -->
+        <origin xyz="0.5 0.0 -0.12" rpy="0.0 0.0 0.0" />
+        <parent link="base_link" />
+        <child link="lidar_mount_link" />
+    </joint>
     <joint name="lidar_link_joint" type="fixed">
-        <origin xyz="0.5 0.0 -0.150" rpy="0.0 -0.0 0.0" />
-        <parent link="base_link" />
+        <!-- Lidar bracket'in ucunda (25cm ileride) -->
+        <origin xyz="0.25 0.0 -0.03" rpy="0.0 0.0 0.0" />
+        <parent link="lidar_mount_link" />
         <child link="lidar_link" />
     </joint>
